Commit message: remove rotors depend

File: urdf/quadrotor_lvi.urdf.xacro (robot description, xacro)
@@ -8,9 +8,15 @@
     <xacro:include filename="$(find velodyne_description)/urdf/VLP-16.urdf.xacro"/>
     <VLP-16 parent="base_link" name="velodyne" topic="/velodyne_points" hz="10" samples="440" gpu="true">
-      <origin xyz="0 0 0.05" rpy="0 0 0" />
+        <origin xyz="0 0 0.05" rpy="0 0 0" />
     </VLP-16>
-    <!-- vi sensor -->
+    <!-- stereo camera -->
+    <xacro:include filename="$(find hector_sensors_description)/urdf/generic_stereo_camera.urdf.xacro"/>
+    <xacro:generic_stereo_camera name="stereo_camera" parent="base_link" ros_topic="image_raw" cam_info_topic="camera_info" update_rate="20.0" res_x="752" res_y="480" image_format="L8" hfov="80.0" baseline="0.11">
+        <origin xyz="0.26 0.055 -0.06" rpy="0 0 0"/>
+    </xacro:generic_stereo_camera>
+    <!--
     <xacro:include filename="$(find rotors_description)/urdf/component_snippets.xacro" />
     <xacro:vi_sensor_stereo_camera_macro namespace="vi_sensor" parent_link="base_link" frame_rate="20.0" origin_offset_x="0.26" baseline_y="${0.055*2}" origin_offset_z="-0.06" max_range="30.0">
     </xacro:vi_sensor_stereo_camera_macro>
+    -->
 </robot>

Commit message: add rgbd camera urdf

File: urdf/quadrotor_lvi.urdf.xacro (robot description, xacro)
@@ -15,8 +15,8 @@
         <origin xyz="0.26 0.055 -0.06" rpy="0 0 0"/>
     </xacro:generic_stereo_camera>
-    <!--
-    <xacro:include filename="$(find rotors_description)/urdf/component_snippets.xacro" />
-    <xacro:vi_sensor_stereo_camera_macro namespace="vi_sensor" parent_link="base_link" frame_rate="20.0" origin_offset_x="0.26" baseline_y="${0.055*2}" origin_offset_z="-0.06" max_range="30.0">
-    </xacro:vi_sensor_stereo_camera_macro>
-    -->
+    <!-- kinect -->
+    <xacro:include filename="$(find my_sim)/urdf/rgbd_camera.urdf.xacro"/>
+    <xacro:rgbd_camera name="kinect" parent="base_link">
+        <origin xyz="0.26 0.055 -0.06" rpy="0 0 0"/>
+    </xacro:rgbd_camera>
 </robot>
